File: schematic/print/print.kicad_sch (KiCad schematic)
At the start: 7 parts, among them U1 LM2575-5.0BT

Commit message: added basic outline, no real values yet
Parts:
- added J1, J2: Conn_01x01, symbol Connector_Generic:Conn_01x01
- added R4: 200k, symbol Device:R
- added R5: 1k, symbol Device:R
- added RShunt: 0.05, symbol Device:R
- added U2: TL084, symbol Amplifier_Operational:TL084
Connections:
- net GND: now also R5.2, RShunt.2
- net at R1.2: now also R2.2, J1.1 (Pin_1)
- new net: R4.2, R5.1, U2.2 (-)
- new net: J2.1 (Pin_1), R4.1, U2.1
- new net I+: RShunt.1, U2.3 (+)

Commit message: added values
Parts:
- removed D1: SB130, Diode_THT:D_DO-41_SOD81_P10.16mm_Horizontal, symbol Diode:SB130
- added D1: IN582, symbol Device:D
- C1: value C -> 470u
- C2: value C -> 220u
- L1: value L -> 440u
- R1: value R -> 52.5k
- R2: value R -> 15k
Connections:
- net GND: now also D1.2 (A)
- net at L1.1, U1.2 (OUT): now also D1.1 (K)
Changed lines of the file:
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@@
+	)
+	(junction
+		(at 129.54 87.63)
+		(diameter 0)
+		(color 0 0 0 0)
 	)
 	(junction
@@
 	)
 	(junction
+		(at 129.54 78.74)
+		(diameter 0)
+		(color 0 0 0 0)
+	)
+	(junction
 		(at 105.41 137.16)
 		(diameter 0)
@@
 	)
 	(junction
-		(at 129.54 88.9)
-		(diameter 0)
-		(color 0 0 0 0)
-	)
-	(junction
 		(at 81.28 87.63)
 		(diameter 0)
@@
 	)
 	(junction
-		(at 129.54 78.74)
-		(diameter 0)
-		(color 0 0 0 0)
-	)
-	(junction
 		(at 114.3 87.63)
 		(diameter 0)
@@
 	(wire
 		(pts
+			(xy 129.54 78.74) (xy 129.54 80.01)
+		)
+		(stroke
+			(width 0)
+			(type default)
+		)
+	)
+	(wire
+		(pts
 			(xy 144.78 86.36) (xy 144.78 88.9)
 		)
@@
 	(wire
 		(pts
+			(xy 129.54 78.74) (xy 133.35 78.74)
+		)
+		(stroke
+			(width 0)
+			(type default)
+		)
+	)
+	(wire
+		(pts
 			(xy 81.28 85.09) (xy 81.28 87.63)
 		)
@@
 	(wire
 		(pts
-			(xy 129.54 78.74) (xy 129.54 81.28)
-		)
-		(stroke
-			(width 0)
-			(type default)
-		)
-	)
-	(wire
-		(pts
 			(xy 87.63 149.86) (xy 97.79 149.86)
 		)
@@
 		(pts
 			(xy 81.28 74.93) (xy 81.28 77.47)
-		)
-		(stroke
-			(width 0)
-			(type default)
-		)
-	)
-	(wire
-		(pts
-			(xy 129.54 78.74) (xy 133.35 78.74)
 		)
 		(stroke
@@
 			)
 		)
-		(property "Value" "R"
+		(property "Value" "52.5k"
 			(at 83.82 97.79 90)
 			(effects
@@
 			)
 		)
-		(property "Value" "R"
+		(property "Value" "15k"
 			(at 83.82 109.22 90)
 			(effects
@@
 			)
 		)
-		(property "Value" "C"
+		(property "Value" "470u"
 			(at 85.09 82.5499 0)
 			(effects
@@
 			)
 		)
-		(property "Value" "C"
+		(property "Value" "220u"
 			(at 148.59 83.8199 0)
 			(effects
@@
 	)
 	(symbol
-		(lib_id "Diode:SB130")
-		(at 129.54 85.09 270)
-		(unit 1)
-		(exclude_from_sim no)
-		(in_bom yes)
-		(on_board yes)
-		(dnp no)
-		(fields_autoplaced yes)
-		(property "Reference" "D1"
-			(at 132.08 83.5024 90)
-			(effects
-				(font
-					(size 1.27 1.27)
-				)
-				(justify left)
-			)
-		)
-		(property "Value" "SB130"
-			(at 132.08 86.0424 90)
-			(effects
-				(font
-					(size 1.27 1.27)
-				)
-				(justify left)
-			)
-		)
-		(property "Footprint" "Diode_THT:D_DO-41_SOD81_P10.16mm_Horizontal"
-			(at 125.095 85.09 0)
-			(effects
-				(font
-					(size 1.27 1.27)
-				)
-				(hide yes)
-			)
-		)
-		(property "Datasheet" "http://www.diodes.com/_files/datasheets/ds23022.pdf"
-			(at 129.54 85.09 0)
-			(effects
-				(font
-					(size 1.27 1.27)
-				)
-				(hide yes)
-			)
-		)
-		(property "Description" "30V 1A Schottky Barrier Rectifier Diode, DO-41"
-			(at 129.54 85.09 0)
-			(effects
-				(font
-					(size 1.27 1.27)
-				)
-				(hide yes)
-			)
-		)
-		(pin "1"
-		)
-		(pin "2"
-		)
-		(instances
-			(project ""
-				(path "/81f2c97a-c73d-48f1-90cd-9aaf7927251a"
-					(reference "D1")
-					(unit 1)
-				)
-			)
-		)
-	)
-	(symbol
 		(lib_id "Device:L")
 		(at 137.16 78.74 90)
@@
 			)
 		)
-		(property "Value" "L"
+		(property "Value" "440u"
 			(at 137.16 76.2 90)
 			(effects
@@
 					(unit 1)
 				)
+			)
+		)
+	)
+	(symbol
+		(lib_id "Device:D")
+		(at 129.54 83.82 270)
+		(unit 1)
+		(exclude_from_sim no)
+		(in_bom yes)
+		(on_board yes)
+		(dnp no)
+		(fields_autoplaced yes)
+		(property "Reference" "D1"
+			(at 132.08 82.5499 90)
+			(effects
+				(font
+					(size 1.27 1.27)
+				)
+				(justify left)
+			)
+		)
+		(property "Value" "IN582"
+			(at 132.08 85.0899 90)
+			(effects
+				(font
+					(size 1.27 1.27)
+				)
+				(justify left)
+			)
+		)
+		(property "Footprint" ""
+			(at 129.54 83.82 0)
+			(effects
+				(font
+					(size 1.27 1.27)
+				)
+				(hide yes)
+			)
+		)
+		(property "Datasheet" "~"
+			(at 129.54 83.82 0)
+			(effects
+				(font
+					(size 1.27 1.27)
+				)
+				(hide yes)
+			)
+		)
+		(property "Description" "Diode"
+			(at 129.54 83.82 0)
+			(effects
+				(font
+					(size 1.27 1.27)
+				)
+				(hide yes)
+			)
+		)
+		(property "Sim.Device" "D"
+			(at 129.54 83.82 0)
+			(effects
+				(font
+					(size 1.27 1.27)
+				)
+				(hide yes)
+			)
+		)
+		(property "Sim.Pins" "1=K 2=A"
+			(at 129.54 83.82 0)
+			(effects
+				(font
+					(size 1.27 1.27)
+				)
+				(hide yes)
+			)
+		)
+		(pin "2"
+		)
+		(pin "1"
+		)
+		(instances
+			(project ""
+				(path "/81f2c97a-c73d-48f1-90cd-9aaf7927251a"
+					(reference "D1")
+					(unit 1)
+				)
